Commit message: Added dockerfile and camera for quadrotor in gazebo

File: quadrotor/urdf/camera.xacro (robot description, xacro)
@@ -12,5 +12,5 @@
     <visual>
       <geometry>
-        <box radius="0.010 0.03 0.03"/>
+        <box size="0.010 0.03 0.03"/>
       </geometry>
       <material name="orange"/>

File: quadrotor/urdf/quadrotor.urdf.xacro (robot description, xacro)
@@ -33,4 +33,5 @@
   <gazebo>
     <plugin name="quadrotor_model" filename="libquadrotor_plugin.so">
+      <max_velocity>0.3</max_velocity>
     </plugin>
   </gazebo>
